File: POWER_DISTRIBUTION/POWER DISTRIBUTIO BOARD_BALLOON/POWER DISTRIBUTIONB BOARD.kicad_pcb (KiCad board)
At the start: 4 copper layers, 94.5 x 55 mm, 98 parts, among them IC3 TPS1HB08BQPWPRQ1, IC4 TPS1HB08BQPWPRQ1, IC8 INA232AIDDFR, IC9 TCAN1044VDDFR, J10 Conn_01x02, J11 Conn_01x02, J28 Conn_01x06, J29 Conn_01x02, J30 Conn_01x02, J31 Conn_01x02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

Commit message: commit after disaster
Parts:
- moved D13 9.27 mm to (166.5, 82.2)
- moved D10 8.80 mm to (175.6, 83.1)
- moved D12 8.80 mm to (182.1, 81.4)
- moved J30 8.80 mm to (181.1, 76.2)
- moved J9 8.80 mm to (172.6, 76.1)
- moved J31 8.80 mm to (165.1, 76.1)
- moved R3 5.33 mm to (185.2, 82.8), turned to -90 degrees
- moved TP27 4.54 mm to (159.6, 80.5)
- moved R5 3.54 mm to (183.5, 82.8), turned to -90 degrees
Routing:
- net GND: track 66.2 -> 52.7 mm, vias 79 -> 74
- net Net-(IC3-LATCH): track 9.26 -> 6.34 mm
