File: POWER_DISTRIBUTION/UREX_PDB/UREX_PDB/PIC.kicad_sch (KiCad schematic)
At the start: 19 parts, among them IC4 INA232AIDDFR

Commit message: FIXED LIBRARY
Parts:
- IC4: footprint SamacSys_Parts_power:SOT65P280X110-8N -> SamacSys_Parts:SOT65P280X110-8N
Other:
- note added: "REMEMBER TO CHECK THAT PIN 4 IS GROUNDED!"
