File: POWER_DISTRIBUTION/UREX_PDB/UREX_PDB/load_switches.kicad_sch (KiCad schematic)
At the start: 28 parts, among them IC2 TPS1HB08BQPWPRQ1, IC3 TPS1HB08BQPWPRQ1, Q1 RSS070N05HZGTB, Q2 RSS070N05HZGTB

Commit message: FIXED LIBRARY
Parts:
- removed D4, D5: SMBJ15CA, SamacSys_Parts:DIOM5436X261N, symbol SamacSys_Parts:SMBJ15CA
- added D6, D9: SMBJ15CA, SamacSys_Parts:DIONM5436X244N, symbol SamacSys_Parts:SMBJ15CA
Connections:
- net GND: now also D6.1, D9.1
- net at Q1.4 (GATE), R43.1: now also D6.2
- net at Q2.4 (GATE), R45.1: now also D9.2
