File: POWER_DISTRIBUTION/UREX_PDB/UREX_PDB/UREX_PDB.kicad_pcb (KiCad board)
At the start: 4 copper layers, 90 x 60 mm, 93 parts, among them IC1 TCAN1044VDDFR, IC2 TPS1HB08BQPWPRQ1, IC3 TPS1HB08BQPWPRQ1, IC4 INA232AIDDFR, J10 Conn_01x02, J11 Conn_01x02, J28 Conn_01x06, J29 Conn_01x02, J30 Conn_01x02, J31 Conn_01x02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

Commit message: FIXED LIBRARY
Parts:
- removed D4, D5: SMBJ15CA, SamacSys_Parts:DIOM5436X261N
- removed J10, J29, J9: Conn_01x02, Connector_JST:JST_PH_S2B-PH-K_1x02_P2.00mm_Horizontal
- removed J30: Conn_01x02, Connector_JST:JST_PH_B2B-PH-K_1x02_P2.00mm_Vertical
- removed J32: Conn_01x04, Connector_JST:JST_PH_S4B-PH-K_1x04_P2.00mm_Horizontal
- removed J35, J36: Conn_01x03, Connector_JST:JST_PH_S3B-PH-K_1x03_P2.00mm_Horizontal
- added D6: SMBJ15CA, SamacSys_Parts:DIONM5436X244N, F.Cu at (65.0, 70.6)
- added D9: SMBJ15CA, SamacSys_Parts:DIONM5436X244N, F.Cu at (65.0, 76.1)
- added J1: S2B-PH-SM4-TB_LF__SN_, SamacSys_Parts:S2BPHSM4TBLFSN, B.Cu at (108.0, 69.2)
- added J13: S2B-PH-SM4-TB_LF__SN_, SamacSys_Parts:S2BPHSM4TBLFSN, F.Cu at (120.5, 132.7)
- added J2: S2B-PH-SM4-TB_LF__SN_, SamacSys_Parts:S2BPHSM4TBLFSN, F.Cu at (48.0, 38.9)
- added J3: S2B-PH-SM4-TB_LF__SN_, SamacSys_Parts:S2BPHSM4TBLFSN, F.Cu at (59.4, 38.9)
- added J5: S3B-PH-SM4-TB_LF__SN_, SamacSys_Parts:S3BPHSM4TBLFSN, B.Cu at (130.0, 69.6)
- added J6: S4B-PH-SM4-TB_LF__SN_, SamacSys_Parts:S4B-PH-SM4-TB, F.Cu at (93.4, 71.6)
- added J7: S2B-PH-SM4-TB_LF__SN_, SamacSys_Parts:S2BPHSM4TBLFSN, F.Cu at (106.6, 139.9)
- added JP3: SolderJumper_2_Open, Jumper:SolderJumper-2_P1.3mm_Open_Pad1.0x1.5mm, B.Cu at (85.8, 101.2)
- added JP4: SolderJumper_2_Open, Jumper:SolderJumper-2_P1.3mm_Open_Pad1.0x1.5mm, B.Cu at (89.6, 101.2)
- C48, J28, J31: moved to B.Cu
- D3: footprint SamacSys_Parts_power:SOT65P210X110-3N -> SamacSys_Parts:SOT65P210X110-3N
- IC1, IC4: footprint SamacSys_Parts_power:SOT65P280X110-8N -> SamacSys_Parts:SOT65P280X110-8N
- J8: value Conn_01x02 -> S3B-PH-SM4-TB_LF__SN_; footprint Connector_JST:JST_PH_S2B-PH-K_1x02_P2.00mm_Horizontal -> SamacSys_Parts:S3BPHSM4TBLFSN; moved to B.Cu
- R45: moved to F.Cu
- moved R56 67.0 mm to (85.0, 88.2), turned to 180 degrees
- moved C53 35.4 mm to (78.1, 50.6)
- moved R58 35.4 mm to (80.5, 51.4)
- moved R59 35.4 mm to (83.7, 51.4)
- moved J8 23.5 mm to (142.6, 69.6), turned to 180 degrees
- moved C52 20.9 mm to (107.4, 80.5)
- moved C51 20.6 mm to (107.5, 78.8)
- moved IC1 19.3 mm to (108.0, 75.9)
- moved J28 9.57 mm to (97.8, 117.2), turned to 180 degrees
- moved C48 8.10 mm to (85.0, 108.8), turned to 0 degrees
- moved C13 4.57 mm to (96.6, 73.8), turned to -90 degrees
- moved C11 4.50 mm to (108.4, 91.7)
- moved C12 4.50 mm to (108.4, 94.7)
- moved C18 4.50 mm to (103.2, 86.5)
- moved C25 4.50 mm to (105.0, 86.5)
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Connections:
- J28 pad 2: CUTTER_EN -> I2C2_SDA
- J28 pad 3: VTX_EN -> I2C2_SDL
- J28 pad 4: I2C2_SDA -> CUTTER_EN_EXT
- J28 pad 5: I2C2_SDL -> VTX_EN_EXT
- J8 pad 1: 12V_BUS2 -> GND
- J8 pad 2: GND -> onewire1
- U7 pad 4: PGM_TX -> PGM_TX_FILT
- U7 pad 6: PGM_RX -> PGM_RX_FILT
Routing:
- net VTX_EN: track 122.9 -> 14.0 mm, vias 3 -> 1
- net BOOT: track 36.9 -> 0.74 mm, vias 2 -> 0
- net onewire1: track 111.5 -> 79.1 mm, vias 3 -> 4
- net CAN-: track 29.1 -> 0.00 mm
- net CAN+: track 28.6 -> 0.00 mm
- net +3V3: track 60.8 -> 34.8 mm, vias 16 -> 14
- net CAN_RX: track 6.75 -> 29.3 mm, vias 0 -> 2
- net CUTTER_EN: track 29.9 -> 7.70 mm, vias 2 -> 1
- net CAN_TX: track 5.94 -> 25.6 mm
- net CUTTER_EN_EXT: track 0.00 -> 17.6 mm
- net VTX_EN_EXT: track 0.00 -> 17.1 mm
- net GND: track 110.3 -> 95.4 mm, vias 170 -> 111
- net onewire2: track 72.5 -> 57.7 mm, vias 1 -> 2
- net Net-(C53-Pad1): track 12.1 -> 0.00 mm, vias 2 -> 0
- net PGM_TX: track 35.7 -> 23.9 mm
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
Commit message: update
Parts:
- removed C53: 4.7nF, Capacitor_SMD:C_0603_1608Metric
- removed D3: PESD2CANFD24V-UX, SamacSys_Parts:SOT65P210X110-3N
- removed J13, J2, J3: S2B-PH-SM4-TB_LF__SN_, SamacSys_Parts:S2BPHSM4TBLFSN
- removed J28: Conn_01x06, Connector_JST:JST_PH_S6B-PH-K_1x06_P2.00mm_Horizontal
- removed J31: Conn_01x02, Connector_JST:JST_PH_S2B-PH-K_1x02_P2.00mm_Horizontal
- removed R58, R59: 60, Resistor_SMD:R_0603_1608Metric
- added J35: Conn_01x02, Connector_JST:JST_PH_S2B-PH-K_1x02_P2.00mm_Horizontal, F.Cu at (125.2, 117.0)
- added J36: Conn_01x02, Connector_JST:JST_PH_S2B-PH-K_1x02_P2.00mm_Horizontal, F.Cu at (165.2, 77.1)
- added J37: Conn_01x02, Connector_JST:JST_PH_S2B-PH-K_1x02_P2.00mm_Horizontal, F.Cu at (165.2, 90.7)
- added J4: S2B-PH-SM4-TB_LF__SN_, SamacSys_Parts:S2BPHSM4TBLFSN, F.Cu at (109.3, 119.0)
- added J9: S6B-PH-SM4-TB_LF__SN_, SamacSys_Parts:S6B-PH-SM4-TB_LF__SN__3, B.Cu at (92.8, 116.3)
- added R2: R_Small, Resistor_SMD:R_0603_1608Metric, B.Cu at (107.9, 76.6)
- C51, C52, D6, D9, IC1, J7: moved to B.Cu
- moved D9 83.8 mm to (141.2, 110.9), turned to -90 degrees
- moved D6 74.4 mm to (128.2, 109.9), turned to -90 degrees
- moved J7 21.1 mm to (109.3, 119.0)
- moved R43 19.2 mm to (124.5, 108.9)
- moved R42 18.3 mm to (124.5, 107.2)
- moved C13 10.6 mm to (91.8, 83.2), turned to 180 degrees
- moved U7 10.3 mm to (88.0, 83.2), turned to 0 degrees
- moved R54 6.35 mm to (97.6, 106.0), turned to 90 degrees
- moved TP6 4.86 mm to (106.3, 110.2)
- moved C18 4.30 mm to (103.2, 90.8)
- moved C25 4.30 mm to (105.0, 90.8)
- moved FB1 4.30 mm to (101.0, 90.7)
- moved PS1 4.30 mm to (108.2, 92.0)
- moved TP5 4.30 mm to (107.3, 87.2)
- moved C51 4.25 mm to (107.4, 83.1), turned to 0 degrees
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Routing:
- net VTX_EN: track 14.0 -> 93.7 mm
- net Net-(Q1-GATE): track 52.7 -> 14.1 mm, vias 2 -> 0
- net HEATER_EN: track 72.6 -> 35.2 mm
- net onewire1: track 79.1 -> 113.0 mm, vias 4 -> 5
- net onewire2: track 57.7 -> 78.5 mm, vias 2 -> 3
- net PGM_TX: track 23.9 -> 11.7 mm
- net PGM_TX_FILT: track 4.95 -> 16.8 mm
- net PGM_RX_FILT: track 4.92 -> 13.6 mm
- net GND: track 95.4 -> 86.7 mm, vias 111 -> 90
- net PGM_RX: track 22.6 -> 15.0 mm, vias 0 -> 2
- net CAN-: track 0.00 -> 7.44 mm
- net CAN+: track 0.00 -> 7.42 mm
- net CAN_RX: track 29.3 -> 22.1 mm, vias 2 -> 1
- net +3V3: track 34.8 -> 28.2 mm, vias 14 -> 20
- net I2C2_SDL: track 55.7 -> 60.4 mm, vias 1 -> 2
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- added copper zone on B.Cu, net +3V3
