File: POWER_DISTRIBUTION/UREX_PDB/UREX_PDB/UREX_PDB.kicad_sch (KiCad schematic)
At the start: 21 parts, among them IC1 TCAN1044VDDFR, J29 Conn_01x02, U6 ESP32-WROOM-32E

Commit message: FIXED LIBRARY
Parts:
- removed J29: Conn_01x02, Connector_JST:JST_PH_S2B-PH-K_1x02_P2.00mm_Horizontal, symbol Connector_Generic:Conn_01x02
- added J1: S2B-PH-SM4-TB_LF__SN_, SamacSys_Parts:S2BPHSM4TBLFSN, symbol SamacSys_Parts:S2B-PH-SM4-TB_LF__SN_
- added JP3, JP4: SolderJumper_2_Open, Jumper:SolderJumper-2_P1.3mm_Open_Pad1.0x1.5mm, symbol Jumper:SolderJumper_2_Open
- D3: footprint SamacSys_Parts_power:SOT65P210X110-3N -> SamacSys_Parts:SOT65P210X110-3N
- IC1: footprint SamacSys_Parts_power:SOT65P280X110-8N -> SamacSys_Parts:SOT65P280X110-8N
Connections:
- net CAN+: now also J1.2
- net CAN-: now also J1.1
- net CUTTER_EN: now also JP4.1 (A)
- net VTX_EN: now also JP3.1 (A)
- new net CUTTER_EN_EXT: JP4.2 (B)
- new net VTX_EN_EXT: JP3.2 (B)
- no-connect marks 15 -> 17

Commit message: update
Parts:
- removed C53: 4.7nF, Capacitor_SMD:C_0603_1608Metric, symbol Device:C_Small
- removed D3: PESD2CANFD24V-UX, SamacSys_Parts:SOT65P210X110-3N, symbol SamacSys_Parts:PESD2CANFD24V-UX
- removed R58, R59: 60, Resistor_SMD:R_0603_1608Metric, symbol Device:R_Small
- added R2: R_Small, Resistor_SMD:R_0603_1608Metric, symbol Device:R_Small
Connections:
- net CAN+: now also R2.1
- net CAN-: now also R2.2
