File: POWER_DISTRIBUTION/UREX_PDB/UREX_PDB/connectors.kicad_sch (KiCad schematic)
At the start: 23 parts, among them J11 Conn_01x02, J33 Conn_01x02, J34 Conn_01x02, J35 Conn_01x02, J36 Conn_01x02, J37 Conn_01x02, J4 S2B-PH-SM4-TB_LF__SN_, J5 S3B-PH-SM4-TB_LF__SN_, J6 S4B-PH-SM4-TB_LF__SN_, J7 S2B-PH-SM4-TB_LF__SN_, J8 S3B-PH-SM4-TB_LF__SN_, J9 S6B-PH-SM4-TB_LF__SN_, U7 USBLC6-2SC6

Commit message: 040722026
Parts:
- removed J35: Conn_01x02, Connector_JST:JST_PH_S2B-PH-K_1x02_P2.00mm_Horizontal, symbol Connector_Generic:Conn_01x02
- added J10: S2B-PH-SM4-TB_LF__SN_, SamacSys_Parts:S2BPHSM4TBLFSN, symbol SamacSys_Parts:S2B-PH-SM4-TB_LF__SN_
- TP2, TP3, TP4, TP5, TP6: footprint TestPoint:TestPoint_Pad_2.0x2.0mm -> SamacSys_Parts:S175146R
Connections:
- net +5V0: now also J10.2
- net GND: now also J10.1
- net PGM_RX_FILT: now also J6.2; no longer J6.3
- net PGM_TX_FILT: now also J6.3; no longer J6.2
- net VBAT_Fused_OUT renamed VBAT_Fused
- no-connect marks 8 -> 10

Commit message: Updated to shift register IC
delete VTX_EN or just do some interrupt
Parts:
- removed D8: SSC53L-E3_57T, SamacSys_Parts:DIOM7959X262N, symbol SamacSys_COMMS:SSC53L-E3_57T
Connections:
- net +5V0 renamed 5VDC_BUS3
- net 5VDC_BUS3: no longer J10.2, J7.2
- new net 5VDC_BUS1: J10.2
- new net 5VDC_BUS2: J7.2

Commit message: LAYOUT FINISHED, DRC NEXT
LESO
Parts:
- added TP7, TP8: TestPoint, TestPoint:TestPoint_THTPad_1.0x1.0mm_Drill0.5mm, symbol Connector:TestPoint
- TP2, TP3, TP4, TP5, TP6: footprint SamacSys_Parts:S175146R -> TestPoint:TestPoint_THTPad_1.0x1.0mm_Drill0.5mm
Connections:
- net 5VDC_BUS1: now also TP7.1
- net 5VDC_BUS2: now also TP8.1
Other:
- moved on the sheet: TP6

Commit message: First Production
Rev1.0 sent for production
Parts:
- TP2, TP3, TP4, TP5, TP6, TP7, TP8: footprint TestPoint:TestPoint_THTPad_1.0x1.0mm_Drill0.5mm -> TestPoint:TestPoint_Pad_1.5x1.5mm
Changed lines of the file:
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@@
 			)
 		)
-		(property "Footprint" "TestPoint:TestPoint_THTPad_1.0x1.0mm_Drill0.5mm"
+		(property "Footprint" "TestPoint:TestPoint_Pad_1.5x1.5mm"
 			(at 40.64 116.84 0)
 			(hide yes)
@@
 			)
 		)
-		(property "Footprint" "TestPoint:TestPoint_THTPad_1.0x1.0mm_Drill0.5mm"
+		(property "Footprint" "TestPoint:TestPoint_Pad_1.5x1.5mm"
 			(at 106.68 54.61 0)
 			(hide yes)
@@
 			)
 		)
-		(property "Footprint" "TestPoint:TestPoint_THTPad_1.0x1.0mm_Drill0.5mm"
+		(property "Footprint" "TestPoint:TestPoint_Pad_1.5x1.5mm"
 			(at 180.34 53.34 0)
 			(hide yes)
@@
 			)
 		)
-		(property "Footprint" "TestPoint:TestPoint_THTPad_1.0x1.0mm_Drill0.5mm"
+		(property "Footprint" "TestPoint:TestPoint_Pad_1.5x1.5mm"
 			(at 31.75 54.61 0)
 			(hide yes)
@@
 			)
 		)
-		(property "Footprint" "TestPoint:TestPoint_THTPad_1.0x1.0mm_Drill0.5mm"
+		(property "Footprint" "TestPoint:TestPoint_Pad_1.5x1.5mm"
 			(at 38.1 26.67 0)
 			(hide yes)
@@
 			)
 		)
-		(property "Footprint" "TestPoint:TestPoint_THTPad_1.0x1.0mm_Drill0.5mm"
+		(property "Footprint" "TestPoint:TestPoint_Pad_1.5x1.5mm"
 			(at 36.83 87.63 0)
 			(hide yes)
@@
 			)
 		)
-		(property "Footprint" "TestPoint:TestPoint_THTPad_1.0x1.0mm_Drill0.5mm"
+		(property "Footprint" "TestPoint:TestPoint_Pad_1.5x1.5mm"
 			(at 40.64 151.13 0)
 			(hide yes)

Commit message: added 5v 8A  dcdc
Parts:
- C13: value 100nF -> 100nF @50V
Changed lines of the file:
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@@
 			)
 		)
-		(property "Value" "100nF"
+		(property "Value" "100nF @50V"
 			(at 104.1463 100.33 90)
 			(show_name no)

Commit message: V1 Full Fabrication(Freezed design)
Parts:
- TP2, TP3, TP4, TP5, TP6, TP7, TP8: footprint TestPoint:TestPoint_Pad_1.5x1.5mm -> TestPoint:TestPoint_Pad_D1.0mm
Changed lines of the file:
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@@
 			)
 		)
-		(property "Footprint" "TestPoint:TestPoint_Pad_1.5x1.5mm"
+		(property "Footprint" "TestPoint:TestPoint_Pad_D1.0mm"
 			(at 40.64 116.84 0)
 			(hide yes)
@@
 			)
 		)
-		(property "Footprint" "TestPoint:TestPoint_Pad_1.5x1.5mm"
+		(property "Footprint" "TestPoint:TestPoint_Pad_D1.0mm"
 			(at 106.68 54.61 0)
 			(hide yes)
@@
 			)
 		)
-		(property "Footprint" "TestPoint:TestPoint_Pad_1.5x1.5mm"
+		(property "Footprint" "TestPoint:TestPoint_Pad_D1.0mm"
 			(at 180.34 53.34 0)
 			(hide yes)
@@
 			)
 		)
-		(property "Footprint" "TestPoint:TestPoint_Pad_1.5x1.5mm"
+		(property "Footprint" "TestPoint:TestPoint_Pad_D1.0mm"
 			(at 31.75 54.61 0)
 			(hide yes)
@@
 			)
 		)
-		(property "Footprint" "TestPoint:TestPoint_Pad_1.5x1.5mm"
+		(property "Footprint" "TestPoint:TestPoint_Pad_D1.0mm"
 			(at 38.1 26.67 0)
 			(hide yes)
@@
 			)
 		)
-		(property "Footprint" "TestPoint:TestPoint_Pad_1.5x1.5mm"
+		(property "Footprint" "TestPoint:TestPoint_Pad_D1.0mm"
 			(at 36.83 87.63 0)
 			(hide yes)
@@
 			)
 		)
-		(property "Footprint" "TestPoint:TestPoint_Pad_1.5x1.5mm"
+		(property "Footprint" "TestPoint:TestPoint_Pad_D1.0mm"
 			(at 40.64 151.13 0)
 			(hide yes)
